File: microbit-right-angle/microbit-right-angle.sch (KiCad schematic (older format))
At the start: 2 parts, among them J1 microbit_edge, J2 microbit_smd_socket

Commit message: Add ncss/oshw logos and URL
Parts:
- added Z1: ncss, logos:ncss, symbol symbol
- added Z2: oshw, logos:OSHW-Logo2_7.3x6mm_Copper, symbol symbol
Changed lines of the file:
@@
 LIBS:microbit-socket
 LIBS:microbit
+LIBS:symbol
 LIBS:microbit-right-angle-cache
 EELAYER 25 0
@@
 Wire Wire Line
 	5750 3300 5950 3300
+$Comp
+L symbol Z1
+U 1 1 5A1EB384
+P 7900 2650
+F 0 "Z1" H 7900 2650 60  0000 C CNN
+F 1 "ncss" H 7900 2450 60  0000 C CNN
+F 2 "logos:ncss" H 7900 2650 60  0001 C CNN
+F 3 "" H 7900 2650 60  0001 C CNN
+	1    7900 2650
+	1    0    0    -1
+$EndComp
+$Comp
+L symbol Z2
+U 1 1 5A1EB3BA
+P 7900 3150
+F 0 "Z2" H 7900 3150 60  0000 C CNN
+F 1 "oshw" H 7900 2950 60  0000 C CNN
+F 2 "logos:OSHW-Logo2_7.3x6mm_Copper" H 7900 3150 60  0001 C CNN
+F 3 "" H 7900 3150 60  0001 C CNN
+	1    7900 3150
+	1    0    0    -1
+$EndComp
 $EndSCHEMATC

Commit message: Update soldermask clearance. Redo big pad connections.
Connections:
- net MB_10: no longer J2.36 (Pin_10_b)
- net MB_3: no longer J2.29 (Pin_3_b)
- net MB_4: no longer J2.30 (Pin_4_b)
- net MB_6: no longer J2.32 (Pin_6_b)
- net MB_7: no longer J2.33 (Pin_7_b)
- net MB_9: no longer J2.35 (Pin_9_b)
- no-connect marks 0 -> 6
Changed lines of the file:
@@
 Text GLabel 4350 4000 0    60   Input ~ 0
 MB_11
-Text GLabel 4350 3900 0    60   Input ~ 0
-MB_10
-Text GLabel 4350 3800 0    60   Input ~ 0
-MB_9
 Text GLabel 4350 3700 0    60   Input ~ 0
 MB_8
-Text GLabel 4350 3600 0    60   Input ~ 0
-MB_7
-Text GLabel 4350 3500 0    60   Input ~ 0
-MB_6
 Text GLabel 4350 3400 0    60   Input ~ 0
 MB_5
-Text GLabel 4350 3300 0    60   Input ~ 0
-MB_4
-Text GLabel 4350 3200 0    60   Input ~ 0
-MB_3
 Text GLabel 4350 3100 0    60   Input ~ 0
 MB_2
@@
 	1    0    0    -1
 $EndComp
+NoConn ~ 4350 3800
+NoConn ~ 4350 3900
+NoConn ~ 4350 3600
+NoConn ~ 4350 3500
+NoConn ~ 4350 3300
+NoConn ~ 4350 3200
 $EndSCHEMATC
